File: cases/plates/kicad/choc/bottom-plate.kicad_pcb (KiCad board)
At the start: 2 copper layers, 243.2 x 136.2 mm, 11 parts

Commit message: updated bottom plate
Parts:
- removed REF** (x9): MountingHole_2.2mm_M2_Pad, MountingHole:MountingHole_2.2mm_M2_Pad
- added ?: , MountingHole:MountingHole_2.2mm_M2_Pad, F.Cu at (224.7, 32.7)
- added ?: , MountingHole:MountingHole_2.2mm_M2_Pad, F.Cu at (93.5, 116.1)
- added ?: , MountingHole:MountingHole_2.2mm_M2_Pad, F.Cu at (123.1, 151.9)
- added ?: , MountingHole:MountingHole_2.2mm_M2_Pad, F.Cu at (178.5, 70.1)
- added ?: , MountingHole:MountingHole_2.2mm_M2_Pad, F.Cu at (167.5, 151.5)
- added ?: , MountingHole:MountingHole_2.2mm_M2_Pad, F.Cu at (48.7, 74.1)
- added ?: , MountingHole:MountingHole_2.2mm_M2_Pad, F.Cu at (240.7, 67.3)
- added ?: , MountingHole:MountingHole_2.2mm_M2_Pad, F.Cu at (113.7, 69.5)
- added ?: , MountingHole:MountingHole_2.2mm_M2_Pad, F.Cu at (198.9, 116.9)
- ?: renamed from REF**; value MountingHole_2.7mm -> (none)
- ?: renamed from REF**; value MountingHole_2.2mm_M2_Pad -> (none)
Routing:
- net DN: track 6.02 -> 0.00 mm
