File: mx/barobord.kicad_pcb (KiCad board)
At the start: 2 copper layers, 243.2 x 136.2 mm, 147 parts, among them J1 Pimoroni, SW1 SW_Push, SW10 SW_Push, SW11 SW_Push, SW12 SW_Push, SW13 SW_Push, SW14 SW_Push, SW15 SW_Push, SW16 SW_Push, SW17 SW_Push, SW18 SW_Push, SW19 SW_Push, SW2 SW_Push, SW20 SW_Push, SW21 SW_Push, SW22 SW_Push, SW23 SW_Push, SW24 SW_Push, SW25 SW_Push, SW26 SW_Push, SW27 SW_Push, SW28 SW_Push, SW29 SW_Push, SW3 SW_Push, SW30 SW_Push, SW31 SW_Push, SW32 SW_Push, SW33 SW_Push, SW34 SW_Push, SW35 SW_Push, SW36 SW_Push, SW37 SW_Push, SW38 SW_Push, SW39 SW_Push, SW4 SW_Push, SW40 SW_Push, SW41 SW_Push, SW42 RotaryEncoder_Switch, SW43 RotaryEncoder_Switch, SW44 EVQWGD001, SW45 EVQWGD001, SW5 SW_Push, SW6 SW_Push, SW7 SW_Push, SW8 SW_Push, SW9 SW_Push, U1 ATmega32U4-A, U2 PRTR5V0U2X, Y1 Crystal_GND24_Small

Commit message: added underglow support for the MX version (not byo-mcu or choc)
Parts:
- added D83: ws2812b, Keebio-Parts:WS2812B, B.Cu at (121.4, 49.3)
- added D84: ws2812b, Keebio-Parts:WS2812B, B.Cu at (64.8, 34.7)
- added D85: ws2812b, Keebio-Parts:WS2812B, B.Cu at (50.3, 75.0)
- added D86: ws2812b, Keebio-Parts:WS2812B, B.Cu at (94.3, 114.6)
- added D87: ws2812b, Keebio-Parts:WS2812B, B.Cu at (125.0, 142.7)
- added D88: ws2812b, Keebio-Parts:WS2812B, B.Cu at (166.0, 142.7)
- added D89: ws2812b, Keebio-Parts:WS2812B, B.Cu at (197.8, 115.3)
- added D90: ws2812b, Keebio-Parts:WS2812B, B.Cu at (244.3, 75.5)
- added D91: ws2812b, Keebio-Parts:WS2812B, B.Cu at (226.7, 35.9)
- added D92: ws2812b, Keebio-Parts:WS2812B, B.Cu at (169.7, 48.7)
- added JP1: Jumper_2_Open, Jumper:SolderJumper-2_P1.3mm_Open_RoundedPad1.0x1.5mm, F.Cu at (133.2, 80.7)
- moved D30 9.70 mm to (251.8, 82.1), turned to 25 degrees
- moved D36 8.59 mm to (175.3, 151.7)
Routing:
- net Net-(D80-Pad2): track 0.00 -> 204.3 mm, vias 0 -> 5
- net Net-(D89-Pad2): track 0.00 -> 83.1 mm, vias 0 -> 4
- net Net-(D85-Pad2): track 0.00 -> 71.2 mm, vias 0 -> 2
- net Net-(D91-Pad2): track 0.00 -> 69.0 mm, vias 0 -> 2
- net Net-(D83-Pad2): track 0.00 -> 61.5 mm, vias 0 -> 2
- net GND: track 1451.0 -> 1503.0 mm, vias 66 -> 76
- net Net-(D88-Pad2): track 0.00 -> 49.9 mm, vias 0 -> 4
- net Net-(D90-Pad2): track 0.00 -> 47.1 mm, vias 0 -> 2
- net Net-(D84-Pad2): track 0.00 -> 46.5 mm
- net Net-(D87-Pad2): track 0.00 -> 41.3 mm, vias 0 -> 2
- net Net-(D86-Pad2): track 0.00 -> 38.6 mm, vias 0 -> 2
- net +5V: track 1454.4 -> 1491.4 mm, vias 64 -> 73
- net row2: track 380.1 -> 391.6 mm
- net Net-(D43-Pad2): track 18.0 -> 22.3 mm, vias 2 -> 4
- net led: track 158.2 -> 155.2 mm
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