File: cases/plates/kicad/barobord-switchplate-outside-pcb.kicad_pcb (KiCad board)
At the start: 2 copper layers, 251 x 144.1 mm, 0 parts

Commit message: updated kicad files according to the previous commit's gerbers
Parts:
- added ?: , MountingHole:MountingHole_2.2mm_M2, F.Cu at (65.4, 128.7)
- added ?: , MountingHole:MountingHole_2.2mm_M2, F.Cu at (113.2, 41.5)
- added ?: , MountingHole:MountingHole_2.2mm_M2, F.Cu at (177.9, 41.5)
- added ?: , MountingHole:MountingHole_2.2mm_M2, F.Cu at (242.0, 26.8)
- added ?: , MountingHole:MountingHole_2.2mm_M2, F.Cu at (268.9, 83.7)
- added ?: , MountingHole:MountingHole_2.2mm_M2, F.Cu at (226.3, 127.5)
- added ?: , MountingHole:MountingHole_2.2mm_M2, F.Cu at (146.0, 163.4)
- added ?: , MountingHole:MountingHole_2.2mm_M2, F.Cu at (22.5, 84.1)
- added ?: , MountingHole:MountingHole_2.2mm_M2, F.Cu at (48.4, 27.1)
Other:
- outline, holes or cut-outs redrawn
