File: byo-mcu/barobord.sch (KiCad schematic (older format))
At the start: 132 parts, among them J1 Pimoroni, SW1 SW_Push, SW10 SW_Push, SW11 SW_Push, SW12 SW_Push, SW13 SW_Push, SW14 SW_Push, SW15 SW_Push, SW16 SW_Push, SW17 SW_Push, SW18 SW_Push, SW19 SW_Push, SW2 SW_Push, SW20 SW_Push, SW21 SW_Push, SW22 SW_Push, SW23 SW_Push, SW24 SW_Push, SW25 SW_Push, SW26 SW_Push, SW27 SW_Push, SW28 SW_Push, SW29 SW_Push, SW3 SW_Push, SW30 SW_Push, SW31 SW_Push, SW32 SW_Push, SW33 SW_Push, SW34 SW_Push, SW35 SW_Push, SW36 SW_Push, SW37 SW_Push, SW38 SW_Push, SW39 SW_Push, SW4 SW_Push, SW40 SW_Push, SW41 SW_Push, SW42 RotaryEncoder_Switch, SW43 RotaryEncoder_Switch, SW44 EVQWGD001, SW45 EVQWGD001, SW5 SW_Push, SW6 SW_Push, SW7 SW_Push, SW8 SW_Push, SW9 SW_Push, U1 Elite-C, U2 nice_nano

Commit message: updated byo-mcu to work
Parts:
- added J2: Conn_01x02_Female, Connector_JST:JST_PH_S2B-PH-K_1x02_P2.00mm_Horizontal, symbol Connector:Conn_01x02_Female
- added SW46: SW_DIP_x01, Button_Switch_THT:SW_CuK_OS102011MA1QN1_SPDT_Angled, symbol Switch:SW_DIP_x01
Connections:
- net ENC2A: now also U1.15 (14/PB3), U2.15 (P1.11); no longer U1.13 (10/PB6), U2.13 (NFC1/P0.09)
- net GND: no longer U1.23 (GND), U2.23 (GND)
- net col3: now also SW43.S1, SW45.S1
- net col4: now also SW42.S1, SW44.S1
- net col5: now also SW10.2
- net col6: now also SW20.2
- net col7: now also SW30.2
- net col8: now also SW40.2
- net row0: now also U1.13 (10/PB6), U2.13 (NFC1/P0.09); no longer D10.1 (K), U1.24 (B0), U2.24 (BATIN/P0.04)
- net row1: no longer D20.1 (K)
- net row2: no longer D30.1 (K), D81.1 (K)
- net row3: no longer D40.1 (K), D82.1 (K)
- removed net col10: SW42.S1, SW43.S1, SW44.S1, SW45.S1, U1.14 (16/PB2), U2.14 (NFC2/P0.10)
- removed net col9: SW10.2, SW20.2, SW30.2, SW40.2, U1.15 (14/PB3), U2.15 (P1.11)
- new net: J2.1 (Pin_1), SW46.2
- new net B+: SW46.1, U1.24 (B0), U2.24 (BATIN/P0.04)
- new net B-: J2.2 (Pin_2), U1.23 (GND), U2.23 (GND)
- new net row4: D10.1 (K), D20.1 (K), D30.1 (K), D40.1 (K), D81.1 (K), D82.1 (K), U1.14 (16/PB2), U2.14 (NFC2/P0.10)
Other:
- moved on the sheet: Brd1, D10, D20, D30, D40, D41, D42, D43, D44, D45, D46, D47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
