File: byo-mcu/choc/barobord.kicad_pcb (KiCad board)
At the start: 2 copper layers, 243.2 x 136.2 mm, 144 parts, among them J1 Pimoroni, J2 Conn_01x02_Female, SW1 SW_Push, SW10 SW_Push, SW11 SW_Push, SW12 SW_Push, SW13 SW_Push, SW14 SW_Push, SW15 SW_Push, SW16 SW_Push, SW17 SW_Push, SW18 SW_Push, SW19 SW_Push, SW2 SW_Push, SW20 SW_Push, SW21 SW_Push, SW22 SW_Push, SW23 SW_Push, SW24 SW_Push, SW25 SW_Push, SW26 SW_Push, SW27 SW_Push, SW28 SW_Push, SW29 SW_Push, SW3 SW_Push, SW30 SW_Push, SW31 SW_Push, SW32 SW_Push, SW33 SW_Push, SW34 SW_Push, SW35 SW_Push, SW36 SW_Push, SW37 SW_Push, SW38 SW_Push, SW39 SW_Push, SW4 SW_Push, SW40 SW_Push, SW41 SW_Push, SW42 RotaryEncoder_Switch, SW43 RotaryEncoder_Switch, SW44 EVQWGD001, SW45 EVQWGD001, SW46 SW_DIP_x01, SW5 SW_Push, SW6 SW_Push, SW7 SW_Push, SW8 SW_Push, SW9 SW_Push, U1 Elite-C, U2 nice_nano

Commit message: converted jst connector from 2 pin to 3 pin to help prevent people from plugging in the battery backwards, and to support both wiring configurations for batteries
Parts:
- removed the ? at (189.8, 123.2)
- removed the ? at (231.6, 73.6)
- removed the ? at (215.6, 39.0)
- removed the ? at (169.4, 76.4)
- removed the ? at (158.4, 157.8)
- removed the ? at (114.0, 158.2)
- removed the ? at (84.4, 121.6)
- removed the ? at (104.6, 75.8)
- removed the ? at (39.6, 80.4)
- added ?: , MountingHole:MountingHole_3.5mm, F.Cu at (177.8, 123.7)
- added ?: , MountingHole:MountingHole_3.5mm, F.Cu at (219.6, 74.1)
- added ?: , MountingHole:MountingHole_3.5mm, F.Cu at (203.6, 39.5)
- added ?: , MountingHole:MountingHole_3.5mm, F.Cu at (157.4, 76.9)
- added ?: , MountingHole:MountingHole_3.5mm, F.Cu at (146.5, 158.3)
- added ?: , MountingHole:MountingHole_3.5mm, F.Cu at (102.0, 158.7)
- added ?: , MountingHole:MountingHole_3.5mm, F.Cu at (72.4, 122.1)
- added ?: , MountingHole:MountingHole_3.5mm, F.Cu at (92.6, 76.3)
- added ?: , MountingHole:MountingHole_3.5mm, F.Cu at (27.7, 80.9)
- J2: value Conn_01x02_Female -> Conn_01x03_Female; footprint Connector_JST:JST_PH_S2B-PH-K_1x02_P2.00mm_Horizontal -> Connector_JST:JST_PH_S3B-PH-K_1x03_P2.00mm_Horizontal
- moved J2 18.4 mm to (64.6, 104.3), turned to 245 degrees
- moved D65 12.0 mm to (150.4, 84.4)
- moved D7 12.0 mm to (166.5, 62.5)
- moved D82 12.0 mm to (146.6, 129.7)
- moved SW16 12.0 mm to (150.4, 84.4)
- moved D63 12.0 mm to (189.0, 122.1)
- moved D66 12.0 mm to (142.4, 67.2)
- moved SW38 12.0 mm to (189.0, 122.1)
- moved SW6 12.0 mm to (142.4, 67.2)
- moved D33 12.0 mm to (61.6, 131.8)
- moved D41 12.0 mm to (34.2, 44.1)
- moved SW1 12.0 mm to (34.2, 44.1)
- moved D72 12.0 mm to (181.7, 61.5)
- moved SW18 12.0 mm to (181.7, 61.5)
- moved D64 12.0 mm to (158.4, 101.6)
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Connections:
- J2 pad 1: Net-(J2-Pad1) -> B-
- J2 pad 2: B- -> Net-(J2-Pad2)
- SW46 pad 2: Net-(J2-Pad1) -> Net-(J2-Pad2)
Routing:
- net Net-(J2-Pad2): track 0.00 -> 83.9 mm, vias 0 -> 1
- net Net-(J2-Pad1): track 75.9 -> 0.00 mm
- net B-: track 111.2 -> 159.1 mm, vias 5 -> 6
- net GND: track 1054.1 -> 1055.0 mm, vias 69 -> 68
Other:
- board text added: "<- Red wire in th middle!"
