File: byo-mcu/mx/barobord.kicad_pcb (KiCad board)
At the start: 2 copper layers, 243.2 x 136.2 mm, 144 parts, among them J1 Pimoroni, J2 Conn_01x02_Female, SW1 SW_Push, SW10 SW_Push, SW11 SW_Push, SW12 SW_Push, SW13 SW_Push, SW14 SW_Push, SW15 SW_Push, SW16 SW_Push, SW17 SW_Push, SW18 SW_Push, SW19 SW_Push, SW2 SW_Push, SW20 SW_Push, SW21 SW_Push, SW22 SW_Push, SW23 SW_Push, SW24 SW_Push, SW25 SW_Push, SW26 SW_Push, SW27 SW_Push, SW28 SW_Push, SW29 SW_Push, SW3 SW_Push, SW30 SW_Push, SW31 SW_Push, SW32 SW_Push, SW33 SW_Push, SW34 SW_Push, SW35 SW_Push, SW36 SW_Push, SW37 SW_Push, SW38 SW_Push, SW39 SW_Push, SW4 SW_Push, SW40 SW_Push, SW41 SW_Push, SW42 RotaryEncoder_Switch, SW43 RotaryEncoder_Switch, SW44 EVQWGD001, SW45 EVQWGD001, SW46 SW_DIP_x01, SW5 SW_Push, SW6 SW_Push, SW7 SW_Push, SW8 SW_Push, SW9 SW_Push, U1 Elite-C, U2 nice_nano

Commit message: converted jst connector from 2 pin to 3 pin to help prevent people from plugging in the battery backwards, and to support both wiring configurations for batteries
Parts:
- removed the ? at (198.9, 116.9)
- removed the ? at (240.7, 67.3)
- removed the ? at (224.7, 32.7)
- removed the ? at (178.4, 70.1)
- removed the ? at (167.5, 151.5)
- removed the ? at (123.1, 151.9)
- removed the ? at (93.4, 115.3)
- removed the ? at (113.7, 69.5)
- removed the ? at (48.7, 74.1)
- added ?: , MountingHole:MountingHole_3.5mm, F.Cu at (192.8, 117.6)
- added ?: , MountingHole:MountingHole_3.5mm, F.Cu at (234.6, 68.0)
- added ?: , MountingHole:MountingHole_3.5mm, F.Cu at (218.6, 33.4)
- added ?: , MountingHole:MountingHole_3.5mm, F.Cu at (172.4, 70.8)
- added ?: , MountingHole:MountingHole_3.5mm, F.Cu at (161.4, 152.2)
- added ?: , MountingHole:MountingHole_3.5mm, F.Cu at (117.0, 152.6)
- added ?: , MountingHole:MountingHole_3.5mm, F.Cu at (87.4, 116.0)
- added ?: , MountingHole:MountingHole_3.5mm, F.Cu at (107.6, 70.2)
- added ?: , MountingHole:MountingHole_3.5mm, F.Cu at (42.6, 74.8)
- J2: value Conn_01x02_Female -> Conn_01x03_Female; footprint Connector_JST:JST_PH_S2B-PH-K_1x02_P2.00mm_Horizontal -> Connector_JST:JST_PH_S3B-PH-K_1x03_P2.00mm_Horizontal
- moved J2 10.8 mm to (81.1, 99.0), turned to 245 degrees
- moved D27 6.11 mm to (182.1, 88.7)
- moved D29 6.11 mm to (216.5, 72.6)
- moved D57 6.11 mm to (106.2, 95.5)
- moved D64 6.11 mm to (173.4, 95.5)
- moved J1 6.11 mm to (139.8, 139.2)
- moved SW25 6.11 mm to (106.2, 95.5)
- moved SW26 6.11 mm to (173.4, 95.5)
- moved SW43 6.11 mm to (151.8, 118.8)
- moved SW45 6.11 mm to (151.8, 118.8)
- moved D28 6.11 mm to (197.2, 76.1)
- moved D39 6.11 mm to (205.2, 93.3)
- moved D40 6.11 mm to (224.5, 89.8)
- moved D52 6.11 mm to (90.1, 85.2)
- moved D53 6.11 mm to (98.1, 68.0)
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Connections:
- J2 pad 1: Net-(J2-Pad1) -> B-
- J2 pad 2: B- -> Net-(J2-Pad2)
- SW46 pad 2: Net-(J2-Pad1) -> Net-(J2-Pad2)
Routing:
- net Net-(J2-Pad2): track 0.00 -> 85.9 mm
- net Net-(J2-Pad1): track 79.9 -> 0.00 mm
- net B-: track 127.2 -> 143.2 mm, vias 5 -> 7
Other:
- board text added: "<- Red wire goes in middle!"
- board text added: "B+"
- board text added: "B-"
